Commit message: prefixed urdf

File: turtlebot2_description/urdf/hexagons.urdf.xacro (robot description, xacro)
@@ -4,16 +4,15 @@
  -->
 <robot name="stack_hexagons" xmlns:xacro="http://ros.org/wiki/xacro">
-  <xacro:include filename="$(find turtlebot2_description)/urdf/common_properties.urdf.xacro"/>
   <!-- Xacro properties -->
   <xacro:property name="M_SCALE" value="0.001"/>
   <!-- Xacro macros -->
   <!-- Pole macros -->
-  <xacro:macro name="stack_bottom_pole" params="parent number x_loc y_loc z_loc roll=0.0 pitch=0.0 yaw=0.0">
+  <xacro:macro name="stack_bottom_pole" params="number x_loc y_loc z_loc roll=0.0 pitch=0.0 yaw=0.0">
     <joint name="pole_bottom_${number}_joint" type="fixed">
       <origin xyz="${x_loc} ${y_loc} ${z_loc}" rpy="${roll} ${pitch} ${yaw}"/>
-      <parent link="${parent}"/>
-      <child link="pole_bottom_${number}_link"/>
-    </joint>
-    <link name="pole_bottom_${number}_link">
+      <parent link="$(arg prefix)base_link"/>
+      <child link="$(arg prefix)pole_bottom_${number}_link"/>
+    </joint>
+    <link name="$(arg prefix)pole_bottom_${number}_link">
       <visual>
         <origin xyz="0 0 0" rpy="0 0 0"/>
@@ -37,11 +36,11 @@
     </link>
   </xacro:macro>
-  <xacro:macro name="stack_middle_pole" params="parent number x_loc y_loc z_loc roll=0.0 pitch=0.0 yaw=0.0">
+  <xacro:macro name="stack_middle_pole" params="number x_loc y_loc z_loc roll=0.0 pitch=0.0 yaw=0.0">
     <joint name="pole_middle_${number}_joint" type="fixed">
       <origin xyz="${x_loc} ${y_loc} ${z_loc}" rpy="${roll} ${pitch} ${yaw}" />
-      <parent link="${parent}"/>
-      <child link="pole_middle_${number}_link"/>
-    </joint>
-    <link name="pole_middle_${number}_link">
+      <parent link="$(arg prefix)base_link"/>
+      <child link="$(arg prefix)pole_middle_${number}_link"/>
+    </joint>
+    <link name="$(arg prefix)pole_middle_${number}_link">
       <visual>
         <origin xyz="0 0 0" rpy="0 ${pi} 0"/>
@@ -65,11 +64,11 @@
     </link>
   </xacro:macro>
-  <xacro:macro name="stack_top_pole" params="parent number x_loc y_loc z_loc roll=0.0 pitch=0.0 yaw=0.0">
+  <xacro:macro name="stack_top_pole" params="number x_loc y_loc z_loc roll=0.0 pitch=0.0 yaw=0.0">
     <joint name="pole_top_${number}_joint" type="fixed">
       <origin xyz="${x_loc} ${y_loc} ${z_loc}" rpy="${roll} ${pitch} ${yaw}"/>
-      <parent link="${parent}"/>
-      <child link="pole_top_${number}_link"/>
-    </joint>
-    <link name="pole_top_${number}_link">
+      <parent link="$(arg prefix)base_link"/>
+      <child link="$(arg prefix)pole_top_${number}_link"/>
+    </joint>
+    <link name="$(arg prefix)pole_top_${number}_link">
       <visual>
         <origin xyz=" 0 0 0" rpy="0 0 0"/>
@@ -93,11 +92,11 @@
     </link>
   </xacro:macro>
-  <xacro:macro name="stack_3d_sensor_pole" params="parent number x_loc y_loc z_loc roll=0.0 pitch=0.0 yaw=0.0">
+  <xacro:macro name="stack_3d_sensor_pole" params="number x_loc y_loc z_loc roll=0.0 pitch=0.0 yaw=0.0">
     <joint name="pole_kinect_${number}_joint" type="fixed">
       <origin xyz="${x_loc} ${y_loc} ${z_loc}" rpy="${roll} ${pitch} ${yaw}"/>
-      <parent link="${parent}"/>
-      <child link="pole_kinect_${number}_link"/>
-    </joint>
-    <link name="pole_kinect_${number}_link">
+      <parent link="$(arg prefix)base_link"/>
+      <child link="$(arg prefix)pole_kinect_${number}_link"/>
+    </joint>
+    <link name="$(arg prefix)pole_kinect_${number}_link">
       <visual>
         <origin xyz="0 0 0" rpy="0 0 0"/>
@@ -122,21 +121,20 @@
   </xacro:macro>
   <!--
-    Stack macro - all the components relative transforms are made with respect
+    Actual stack - all the components relative transforms are made with respect
     to the parent link (usually base_link). They could be made relative to each
     other, but there is no necessary reason to do so.
   -->
-  <xacro:macro name="stack_hexagons" params="parent">
-    <xacro:stack_bottom_pole parent="${parent}" number="0" x_loc= "0.120" y_loc= "0.082" z_loc="0.1028"/>
-    <xacro:stack_bottom_pole parent="${parent}" number="1" x_loc= "0.055" y_loc= "0.120" z_loc="0.1028"/>
-    <xacro:stack_bottom_pole parent="${parent}" number="2" x_loc="-0.055" y_loc= "0.120" z_loc="0.1028"/>
-    <xacro:stack_bottom_pole parent="${parent}" number="3" x_loc= "0.120" y_loc="-0.082" z_loc="0.1028"/>
-    <xacro:stack_bottom_pole parent="${parent}" number="4" x_loc= "0.055" y_loc="-0.120" z_loc="0.1028"/>
-    <xacro:stack_bottom_pole parent="${parent}" number="5" x_loc="-0.055" y_loc="-0.120" z_loc="0.1028"/>
+    <xacro:stack_bottom_pole number="0" x_loc= "0.120" y_loc= "0.082" z_loc="0.1028"/>
+    <xacro:stack_bottom_pole number="1" x_loc= "0.055" y_loc= "0.120" z_loc="0.1028"/>
+    <xacro:stack_bottom_pole number="2" x_loc="-0.055" y_loc= "0.120" z_loc="0.1028"/>
+    <xacro:stack_bottom_pole number="3" x_loc= "0.120" y_loc="-0.082" z_loc="0.1028"/>
+    <xacro:stack_bottom_pole number="4" x_loc= "0.055" y_loc="-0.120" z_loc="0.1028"/>
+    <xacro:stack_bottom_pole number="5" x_loc="-0.055" y_loc="-0.120" z_loc="0.1028"/>
     <joint name="plate_bottom_joint" type="fixed">
       <origin xyz="0.02364 0.0 0.1306" rpy="0 0 0"/>
-      <parent link="${parent}"/>
-      <child link="plate_bottom_link"/>
-    </joint>
-    <link name="plate_bottom_link">
+      <parent link="$(arg prefix)base_link"/>
+      <child link="$(arg prefix)plate_bottom_link"/>
+    </joint>
+    <link name="$(arg prefix)plate_bottom_link">
       <visual>
         <origin xyz="0 0 0" rpy="0 0 0"/>
@@ -159,14 +157,14 @@
       </inertial>
     </link>
-    <xacro:stack_middle_pole parent="${parent}" number="0" x_loc= "0.0381" y_loc= "0.1505" z_loc="0.1640"/>
-    <xacro:stack_middle_pole parent="${parent}" number="1" x_loc= "0.0381" y_loc="-0.1505" z_loc="0.1640"/>
-    <xacro:stack_middle_pole parent="${parent}" number="2" x_loc="-0.0381" y_loc= "0.1505" z_loc="0.1640"/>
-    <xacro:stack_middle_pole parent="${parent}" number="3" x_loc="-0.0381" y_loc="-0.1505" z_loc="0.1640"/>
+    <xacro:stack_middle_pole number="0" x_loc= "0.0381" y_loc= "0.1505" z_loc="0.1640"/>
+    <xacro:stack_middle_pole number="1" x_loc= "0.0381" y_loc="-0.1505" z_loc="0.1640"/>
+    <xacro:stack_middle_pole number="2" x_loc="-0.0381" y_loc= "0.1505" z_loc="0.1640"/>
+    <xacro:stack_middle_pole number="3" x_loc="-0.0381" y_loc="-0.1505" z_loc="0.1640"/>
     <joint name="plate_middle_joint" type="fixed">
       <origin xyz="-0.01364 0.0 0.1874" rpy="0 0 0"/>
-      <parent link="${parent}"/>
-      <child link="plate_middle_link"/>
-    </joint>
-    <link name="plate_middle_link">
+      <parent link="$(arg prefix)base_link"/>
+      <child link="$(arg prefix)plate_middle_link"/>
+    </joint>
+    <link name="$(arg prefix)plate_middle_link">
       <visual>
         <origin xyz="0 0 0" rpy="0 0 0"/>
@@ -190,16 +188,16 @@
       </inertial>
     </link>
-    <xacro:stack_top_pole parent="${parent}" number="0" x_loc= "0.0381" y_loc= "0.1505" z_loc="0.2920"/>
-    <xacro:stack_top_pole parent="${parent}" number="1" x_loc= "0.0381" y_loc="-0.1505" z_loc="0.2920"/>
-    <xacro:stack_top_pole parent="${parent}" number="2" x_loc="-0.0381" y_loc= "0.1505" z_loc="0.2920"/>
-    <xacro:stack_top_pole parent="${parent}" number="3" x_loc="-0.0381" y_loc="-0.1505" z_loc="0.2920"/>
-    <xacro:stack_3d_sensor_pole parent="${parent}" number="0" x_loc="-0.1024" y_loc= "0.098" z_loc="0.2372"/>
-    <xacro:stack_3d_sensor_pole parent="${parent}" number="1" x_loc="-0.1024" y_loc="-0.098" z_loc="0.2372"/>
+    <xacro:stack_top_pole number="0" x_loc= "0.0381" y_loc= "0.1505" z_loc="0.2920"/>
+    <xacro:stack_top_pole number="1" x_loc= "0.0381" y_loc="-0.1505" z_loc="0.2920"/>
+    <xacro:stack_top_pole number="2" x_loc="-0.0381" y_loc= "0.1505" z_loc="0.2920"/>
+    <xacro:stack_top_pole number="3" x_loc="-0.0381" y_loc="-0.1505" z_loc="0.2920"/>
+    <xacro:stack_3d_sensor_pole number="0" x_loc="-0.1024" y_loc= "0.098" z_loc="0.2372"/>
+    <xacro:stack_3d_sensor_pole number="1" x_loc="-0.1024" y_loc="-0.098" z_loc="0.2372"/>
     <joint name="plate_top_joint" type="fixed">
       <origin xyz="-0.01364 0.0  0.3966" rpy="0 0 0"/>
-      <parent link="${parent}"/>
-      <child link="plate_top_link"/>
-    </joint>
-    <link name="plate_top_link">
+      <parent link="$(arg prefix)base_link"/>
+      <child link="$(arg prefix)plate_top_link"/>
+    </joint>
+    <link name="$(arg prefix)plate_top_link">
       <visual>
         <origin xyz="0 0 0" rpy="0 0 0"/>
@@ -223,4 +221,3 @@
       </inertial>
     </link>
-  </xacro:macro>
 </robot>

File: turtlebot2_description/urdf/kobuki.urdf.xacro (robot description, xacro)
@@ -1,11 +1,5 @@
 <?xml version="1.0" ?>
-<!--
-  This is not a standalone urdf for kobuki. It simply defines the 'kobuki' tag that can
-  be incorporated by other urdf files (e.g. turtlebot).
-  See kobuki_standalone.urdf.xacro for a standalone urdf to be tested with
-      kobuki_description/launch/view_model.launch
- -->
 <robot name="kobuki" xmlns:xacro="http://ros.org/wiki/xacro">
-    <link name="base_footprint"/>
+    <link name="$(arg prefix)base_footprint"/>
     <!--
        Base link is set at the bottom of the base mould.
@@ -19,8 +13,8 @@
     <joint name="base_joint" type="fixed">
       <origin xyz="0 0 0.0102" rpy="0 0 0" />
-      <parent link="base_footprint"/>
-      <child link="base_link" />
-    </joint>
-    <link name="base_link">
+      <parent link="$(arg prefix)base_footprint"/>
+      <child link="$(arg prefix)base_link" />
+    </joint>
+    <link name="$(arg prefix)base_link">
       <visual>
         <geometry>
@@ -40,5 +34,5 @@
         <origin xyz="0.01 0 0"/>
         <mass value="2.4"/> <!-- 2.4/2.6 kg for small/big battery pack -->
-        <!-- Kobuki's inertia tensor is approximated by a cylinder with homogeneous mass distribution
+        <!-- Kobuki inertia tensor is approximated by a cylinder with homogeneous mass distribution
              More details http://en.wikipedia.org/wiki/List_of_moment_of_inertia_tensors
              m = 2.4 kg; h = 0.09 m; r = 0.175 m
@@ -53,10 +47,10 @@
     </link>
     <joint name="wheel_left_joint" type="continuous">
-      <parent link="base_link"/>
-      <child link="wheel_left_link"/>
+      <parent link="$(arg prefix)base_link"/>
+      <child link="$(arg prefix)wheel_left_link"/>
       <origin xyz="0.00 ${0.23/2} 0.0250" rpy="${-pi/2} 0 0"/>
       <axis xyz="0 0 1"/>
     </joint>
-    <link name="wheel_left_link">
+    <link name="$(arg prefix)wheel_left_link">
       <visual>
         <geometry>
@@ -80,10 +74,10 @@
     </link>
     <joint name="wheel_right_joint" type="continuous">
-      <parent link="base_link"/>
-      <child link="wheel_right_link"/>
+      <parent link="$(arg prefix)base_link"/>
+      <child link="$(arg prefix)wheel_right_link"/>
       <origin xyz="0.00 -${0.23/2} 0.0250" rpy="${-pi/2} 0 0"/>
       <axis xyz="0 0 1"/>
     </joint>
-    <link name="wheel_right_link">
+    <link name="$(arg prefix)wheel_right_link">
       <visual>
         <geometry>
@@ -107,9 +101,9 @@
     </link>
     <joint name="caster_front_joint" type="fixed">
-      <parent link="base_link"/>
-      <child link="caster_front_link"/>
+      <parent link="$(arg prefix)base_link"/>
+      <child link="$(arg prefix)caster_front_link"/>
       <origin xyz="0.115 0.0 0.007" rpy="${-pi/2} 0 0"/>
     </joint>
-    <link name="caster_front_link">
+    <link name="$(arg prefix)caster_front_link">
       <collision>
         <geometry>
@@ -127,9 +121,9 @@
     </link>
     <joint name="caster_back_joint" type="fixed">
-      <parent link="base_link"/>
-      <child link="caster_back_link"/>
+      <parent link="$(arg prefix)base_link"/>
+      <child link="$(arg prefix)caster_back_link"/>
       <origin xyz="-0.135 0.0 0.009" rpy="${-pi/2} 0 0"/>
     </joint>
-    <link name="caster_back_link">
+    <link name="$(arg prefix)caster_back_link">
       <collision>
         <geometry>
@@ -146,12 +140,12 @@
       </inertial>
     </link>
-    <!-- Kobuki's sensors -->
+    <!-- sensors -->
     <joint name="gyro_joint" type="fixed">
       <axis xyz="0 1 0"/>
       <origin xyz="0.056 0.062 0.0202" rpy="0 0 0"/>
-      <parent link="base_link"/>
-      <child link="gyro_link"/>
-    </joint>
-    <link name="gyro_link">
+      <parent link="$(arg prefix)base_link"/>
+      <child link="$(arg prefix)gyro_link"/>
+    </joint>
+    <link name="$(arg prefix)gyro_link">
       <inertial>
         <mass value="0.001"/>
@@ -164,8 +158,8 @@
     <joint name="cliff_sensor_left_joint" type="fixed">
       <origin xyz="0.08734 0.13601 0.0214" rpy="0 ${pi/2} 0" />
-      <parent link="base_link"/>
-      <child link="cliff_sensor_left_link" />
-    </joint>
-    <link name="cliff_sensor_left_link">
+      <parent link="$(arg prefix)base_link"/>
+      <child link="$(arg prefix)cliff_sensor_left_link" />
+    </joint>
+    <link name="$(arg prefix)cliff_sensor_left_link">
       <inertial>
         <mass value="0.0001" />
@@ -178,8 +172,8 @@
     <joint name="cliff_sensor_right_joint" type="fixed">
       <origin xyz="0.085 -0.13601 0.0214" rpy="0 ${pi/2} 0" />
-      <parent link="base_link"/>
-      <child link="cliff_sensor_right_link" />
-    </joint>
-    <link name="cliff_sensor_right_link">
+      <parent link="$(arg prefix)base_link"/>
+      <child link="$(arg prefix)cliff_sensor_right_link" />
+    </joint>
+    <link name="$(arg prefix)cliff_sensor_right_link">
       <inertial>
         <mass value="0.0001" />
@@ -192,8 +186,8 @@
     <joint name="cliff_sensor_front_joint" type="fixed">
       <origin xyz="0.156 0.00 0.0214" rpy="0 ${pi/2} 0" />
-      <parent link="base_link"/>
-      <child link="cliff_sensor_front_link" />
-    </joint>
-    <link name="cliff_sensor_front_link">
+      <parent link="$(arg prefix)base_link"/>
+      <child link="$(arg prefix)cliff_sensor_front_link" />
+    </joint>
+    <link name="$(arg prefix)cliff_sensor_front_link">
       <inertial>
         <mass value="0.0001" />

File: turtlebot2_description/urdf/sensors/hokuyo.urdf.xacro (robot description, xacro)
@@ -1,11 +1,7 @@
 <?xml version="1.0"?>
 <robot name="sensor_hokuyo" xmlns:xacro="http://ros.org/wiki/xacro">
-    <xacro:include filename="$(find turtlebot2_description)/urdf/turtlebot_gazebo.urdf.xacro" />
-    <xacro:include filename="$(find turtlebot2_description)/urdf/turtlebot_properties.urdf.xacro" />
-    <xacro:property name="laser_px" value="0.1" />
+    <xacro:property name="laser_px" value="0." />
     <xacro:property name="laser_py" value="0" />
-    <xacro:property name="laser_pz" value="0.21" />
-    <xacro:arg name="namespace" default=""/>
-    <xacro:property name="robot_namespace" value="/$(arg namespace)"/>
+    <xacro:property name="laser_pz" value="0.43" />
     <xacro:macro name="box_inertia" params="x y z mass">
         <inertia ixx="${0.0833333 * mass * (y*y + z*z)}" ixy="0.0" ixz="0.0" iyy="${0.0833333 * mass * (x*x + z*z)}" iyz="0.0" izz="${0.0833333 * mass * (x*x + y*y)}" />
@@ -14,11 +10,10 @@
         <color rgba="1.0 0.423529411765 0.0392156862745 1.0" />
     </material>
-    <xacro:macro name="sensor_hokuyo" params="parent">
         <joint name="laser_joint" type="fixed">
             <origin xyz="${laser_px} ${laser_py} ${laser_pz}" rpy="0 0 0" />
-            <parent link="${parent}" />
-            <child link="laser" />
+            <parent link="$(arg prefix)base_footprint" />
+            <child link="$(arg prefix)laser" />
         </joint>
-        <link name="laser">
+        <link name="$(arg prefix)laser">
             <inertial>
                 <origin xyz="0 0 0" rpy="0 0 0" />
@@ -40,5 +35,6 @@
             </collision>
         </link>
-        <gazebo reference="laser">
+<xacro:if value="$(arg gazebo)">
+        <gazebo reference="$(arg prefix)laser">
             <sensor type="ray" name="head_hokuyo_sensor">
                 <pose>0 0 0 0 0 0</pose>
@@ -80,4 +76,4 @@
             <material>Gazebo/Orange</material>
         </gazebo>
-    </xacro:macro>
+    </xacro:if>
 </robot>

File: turtlebot2_description/urdf/sensors/kinect.urdf.xacro (robot description, xacro)
@@ -1,31 +1,27 @@
 <?xml version="1.0"?>
 <robot name="sensor_kinect" xmlns:xacro="http://ros.org/wiki/xacro">
-  <xacro:include filename="$(find turtlebot_description)/urdf/turtlebot_gazebo.urdf.xacro"/>
-  <xacro:include filename="$(find turtlebot_description)/urdf/turtlebot_properties.urdf.xacro"/>
   <xacro:property name="kinect_cam_py" value="-0.0125"/>
-  <!-- Parameterised in part by the values in turtlebot_properties.urdf.xacro -->
-  <xacro:macro name="sensor_kinect" params="parent">
     <joint name="camera_rgb_joint" type="fixed">
       <origin xyz="${cam_px} ${kinect_cam_py} ${cam_pz}" rpy="${cam_or} ${cam_op} ${cam_oy}"/>
-      <parent link="${parent}"/>
-      <child link="camera_rgb_frame" />
+      <parent link="$(arg prefix)base_link"/>
+      <child link="$(arg prefix)camera_rgb_frame" />
     </joint>
-    <link name="camera_rgb_frame"/>
+    <link name="$(arg prefix)camera_rgb_frame"/>
     <joint name="camera_rgb_optical_joint" type="fixed">
       <origin xyz="0 0 0" rpy="${-pi/2} 0 ${-pi/2}" />
-      <parent link="camera_rgb_frame" />
-      <child link="camera_rgb_optical_frame" />
+      <parent link="$(arg prefix)camera_rgb_frame" />
+      <child link="$(arg prefix)camera_rgb_optical_frame" />
     </joint>
-    <link name="camera_rgb_optical_frame"/>
+    <link name="$(arg prefix)camera_rgb_optical_frame"/>
     <joint name="camera_joint" type="fixed">
       <origin xyz="-0.031 ${-kinect_cam_py} -0.016" rpy="0 0 0"/>
-      <parent link="camera_rgb_frame"/>
-      <child link="camera_link"/>
+      <parent link="$(arg prefix)camera_rgb_frame"/>
+      <child link="$(arg prefix)camera_link"/>
     </joint>
-      <link name="camera_link">
+      <link name="$(arg prefix)camera_link">
       <visual>
        <origin xyz="0 0 0" rpy="0 0 ${pi/2}"/>
         <geometry>
-         <mesh filename="package://turtlebot_description/meshes/sensors/kinect.dae"/>
+         <mesh filename="package://turtlebot2_description/meshes/sensors/kinect.dae"/>
         </geometry>
       </visual>
@@ -46,19 +42,16 @@
     <!-- The fixed joints & links below are usually published by static_transformers launched by the OpenNi launch
          files. However, for Gazebo simulation we need them, so we add them here.
-         (Hence, don't publish them additionally!) -->
+         (Hence, dont publish them additionally!) -->
 	<joint name="camera_depth_joint" type="fixed">
 	  <origin xyz="0 ${2 * -kinect_cam_py} 0" rpy="0 0 0" />
-	  <parent link="camera_rgb_frame" />
-	  <child link="camera_depth_frame" />
+	  <parent link="$(arg prefix)camera_rgb_frame" />
+	  <child link="$(arg prefix)camera_depth_frame" />
 	</joint>
-	<link name="camera_depth_frame"/>
+	<link name="$(arg prefix)camera_depth_frame"/>
 	<joint name="camera_depth_optical_joint" type="fixed">
 	  <origin xyz="0 0 0" rpy="${-pi/2} 0 ${-pi/2}" />
-	  <parent link="camera_depth_frame" />
-	  <child link="camera_depth_optical_frame" />
+	  <parent link="$(arg prefix)camera_depth_frame" />
+	  <child link="$(arg prefix)camera_depth_optical_frame" />
 	</joint>
-	<link name="camera_depth_optical_frame"/>
-	<!-- Kinect sensor for simulation -->
-	<xacro:turtlebot_sim_3dsensor/>
-  </xacro:macro>
+	<link name="$(arg prefix)camera_depth_optical_frame"/>
 </robot>

File: turtlebot2_description/urdf/turtlebot2.urdf.xacro (robot description, xacro)
@@ -4,19 +4,5 @@
   <xacro:arg name="gazebo"  default="false"/>
   <xacro:arg name="hokuyo"  default="true"/>
-  <xacro:arg name="rgbd"    default="kinect"/> <!-- kinect / -->
- <xacro:macro name="mesh" params="pkg mesh">
-      <xacro:if value="${pkg == 'kobuki_description'}">
-        <xacro:property name="scale" value="1." />
-      </xacro:if>
-      <xacro:if value="${pkg == 'turtlebot2_description'}">
-        <xacro:property name="scale" value="0.001" />
-      </xacro:if>
-   <xacro:if value="$(arg gazebo)">
-     <mesh filename="file://$(find ${pkg})/meshes/${mesh}" scale="${scale} ${scale} ${scale}"/>
-   </xacro:if>
-   <xacro:unless value="$(arg gazebo)">
-     <mesh filename="package://turtlebot2_description/meshes/${mesh}" scale="${scale} ${scale} ${scale}"/>
-   </xacro:unless>
- </xacro:macro>
+  <xacro:arg name="kinect"    default="true"/>
   <xacro:include filename="$(find turtlebot2_description)/urdf/common/common_properties.urdf.xacro" />
   <xacro:include filename="$(find turtlebot2_description)/urdf/common/turtlebot_properties.urdf.xacro" />
@@ -26,7 +12,6 @@
     <xacro:include filename="$(find turtlebot2_description)/urdf/sensors/hokuyo.urdf.xacro" />
   </xacro:if>
-  <xacro:if value="$(arg gazebo)">
-   <xacro:include filename="$(find turtlebot2_description)/urdf/gazebo.xacro"/>
+  <xacro:if value="$(arg kinect)">
+    <xacro:include filename="$(find turtlebot2_description)/urdf/sensors/kinect.urdf.xacro"/>
   </xacro:if>
-  <xacro:include filename="$(find turtlebot_description)/urdf/sensors/kinect.urdf.xacro"/>
 </robot>
