Commit message: kobuki + hokuyo plugins for Gazebo Sim

File: turtlebot2_description/urdf/kobuki.urdf.xacro (robot description, xacro)
@@ -198,3 +198,116 @@
       </inertial>
     </link>
+<xacro:if value="$(arg gazebo)">
+<gazebo reference="$(arg prefix)wheel_left_link">
+  <mu1>0.1</mu1>
+  <mu2>0.1</mu2>
+  <kp>500000.0</kp>
+  <kd>10.0</kd>
+  <minDepth>0.001</minDepth>
+  <maxVel>0.1</maxVel>
+  <fdir1>1 0 0</fdir1>
+  <material>Gazebo/FlatBlack</material>
+</gazebo>
+<gazebo reference="$(arg prefix)wheel_right_link">
+  <mu1>0.1</mu1>
+  <mu2>0.1</mu2>
+  <kp>500000.0</kp>
+  <kd>10.0</kd>
+  <minDepth>0.001</minDepth>
+  <maxVel>0.1</maxVel>
+  <fdir1>1 0 0</fdir1>
+  <material>Gazebo/FlatBlack</material>
+</gazebo>
+<gazebo reference="$(arg prefix)caster_back_right_link">
+  <mu1>0.1</mu1>
+  <mu2>0.1</mu2>
+  <kp>1000000.0</kp>
+  <kd>100.0</kd>
+  <minDepth>0.001</minDepth>
+  <maxVel>1.0</maxVel>
+  <material>Gazebo/FlatBlack</material>
+</gazebo>
+<gazebo reference="$(arg prefix)caster_back_left_link">
+  <mu1>0.1</mu1>
+  <mu2>0.1</mu2>
+  <kp>1000000.0</kp>
+  <kd>100.0</kd>
+  <minDepth>0.001</minDepth>
+  <maxVel>1.0</maxVel>
+  <material>Gazebo/FlatBlack</material>
+</gazebo>
+  <gazebo reference="$(arg prefix)gyro_link">
+    <sensor name="tb2_imu" type="imu">
+        <always_on>true</always_on>
+        <update_rate>50</update_rate>
+        <topic>$(arg prefix)imu</topic>
+        <gz_frame_id>$(arg prefix)gyro_link</gz_frame_id>
+        <imu>
+          <angular_velocity>
+            <x>
+              <noise type="gaussian">
+                <mean>0.0</mean>
+                <stddev>2e-4</stddev>
+              </noise>
+            </x>
+            <y>
+              <noise type="gaussian">
+                <mean>0.0</mean>
+                <stddev>2e-4</stddev>
+              </noise>
+            </y>
+            <z>
+              <noise type="gaussian">
+                <mean>0.0</mean>
+                <stddev>2e-4</stddev>
+              </noise>
+            </z>
+          </angular_velocity>
+          <linear_acceleration>
+            <x>
+              <noise type="gaussian">
+                <mean>0.0</mean>
+                <stddev>1.7e-2</stddev>
+              </noise>
+            </x>
+            <y>
+              <noise type="gaussian">
+                <mean>0.0</mean>
+                <stddev>1.7e-2</stddev>
+              </noise>
+            </y>
+            <z>
+              <noise type="gaussian">
+                <mean>0.0</mean>
+                <stddev>1.7e-2</stddev>
+              </noise>
+            </z>
+          </linear_acceleration>
+        </imu>
+    </sensor>
+    <material>Gazebo/Grey</material>
+  </gazebo>
+ <gazebo>
+    <plugin
+      filename="libignition-gazebo-diff-drive-system.so"
+      name="ignition::gazebo::systems::DiffDrive">
+      <left_joint>wheel_left_joint</left_joint>
+      <right_joint>wheel_right_joint</right_joint>
+      <wheel_separation>0.230</wheel_separation>
+      <wheel_radius>0.035</wheel_radius>
+      <child_frame_id>$(arg prefix)base_footprint</child_frame_id>
+      <max_wheel_torque>1.0</max_wheel_torque>
+      <max_wheel_acceleration>1.0</max_wheel_acceleration>
+    </plugin>
+    <plugin filename="libignition-gazebo-joint-state-publisher-system.so" name="ignition::gazebo::systems::JointStatePublisher"/>
+      <plugin
+            filename="ignition-gazebo-pose-publisher-system"
+            name="ignition::gazebo::systems::PosePublisher">
+            <publish_link_pose>false</publish_link_pose>
+            <publish_collision_pose>false</publish_collision_pose>
+            <publish_visual_pose>false</publish_visual_pose>
+            <publish_nested_model_pose>true</publish_nested_model_pose>
+        </plugin>
+</gazebo>
+</xacro:if>
 </robot>

File: turtlebot2_description/urdf/sensors/hokuyo.urdf.xacro (robot description, xacro)
@@ -36,44 +36,35 @@
         </link>
 <xacro:if value="$(arg gazebo)">
-        <gazebo reference="$(arg prefix)laser">
-            <sensor type="ray" name="head_hokuyo_sensor">
-                <pose>0 0 0 0 0 0</pose>
-                <visualize>false</visualize>
-                <update_rate>20</update_rate>
-                <ray>
-                    <scan>
-                        <horizontal>
-                            <samples>720</samples>
-                            <resolution>1</resolution>
-                            <!-- <min_angle>-2.355</min_angle>
-                            <max_angle>2.355</max_angle> -->
-                            <min_angle>-1.56</min_angle>
-                            <max_angle>1.56</max_angle>
-                        </horizontal>
-                    </scan>
-                    <range>
-                        <min>0.10</min>
-                        <max>10.0</max>
-                        <resolution>0.01</resolution>
-                    </range>
-                    <noise>
-                        <type>gaussian</type>
-                        <mean>0.0</mean>
-                        <stddev>0.01</stddev>
-                    </noise>
-                </ray>
-                <plugin name="turtlebot2_laserscan" filename="libgazebo_ros_ray_sensor.so">
-                    <ros>
-                      <remapping>~/out:=scan</remapping>
-		              <namespace>${robot_namespace}</namespace>
-                    </ros>
-                    <output_type>sensor_msgs/LaserScan</output_type>
-                    <frame_name>laser</frame_name>
-                  </plugin>
-            </sensor>
-        </gazebo>
-        <gazebo reference="laser">
-            <material>Gazebo/Orange</material>
-        </gazebo>
+      <gazebo reference="$(arg prefix)laser">
+    <material>Gazebo/FlatBlack</material>
+    <sensor type="gpu_ray" name="head_hokuyo_sensor">
+<!--       <pose>0 0 0 0 0 0</pose> -->
+      <update_rate>20</update_rate>
+      <topic>$(arg prefix)scan</topic>
+      <gz_frame_id>$(arg prefix)laser</gz_frame_id>
+      <ray>
+        <scan>
+            <horizontal>
+                <samples>720</samples>
+                <resolution>1</resolution>
+                <!-- <min_angle>-2.355</min_angle>
+                <max_angle>2.355</max_angle> -->
+                <min_angle>-1.56</min_angle>
+                <max_angle>1.56</max_angle>
+            </horizontal>
+        </scan>
+        <range>
+            <min>0.10</min>
+            <max>10.0</max>
+            <resolution>0.01</resolution>
+        </range>
+        <noise>
+          <type>gaussian</type>
+          <mean>0.0</mean>
+          <stddev>0.01</stddev>
+        </noise>
+      </ray>
+    </sensor>
+  </gazebo>
     </xacro:if>
 </robot>

File: turtlebot2_description/urdf/sensors/kinect.urdf.xacro (robot description, xacro)
@@ -55,3 +55,41 @@
 	</joint>
 	<link name="$(arg prefix)camera_depth_optical_frame"/>
+      <xacro:macro name="turtlebot_sim_3dsensor">
+    <gazebo reference="camera_link">
+      <sensor type="depth" name="camera">
+        <always_on>true</always_on>
+        <update_rate>20.0</update_rate>
+        <camera>
+          <horizontal_fov>${60.0*pi/180.0}</horizontal_fov>
+          <image>
+            <format>B8G8R8</format>
+            <width>640</width>
+            <height>480</height>
+          </image>
+          <clip>
+            <near>0.05</near>
+            <far>8.0</far>
+          </clip>
+        </camera>
+        <plugin name="kinect_camera_controller" filename="libgazebo_ros_openni_kinect.so">
+          <cameraName>camera</cameraName>
+          <alwaysOn>true</alwaysOn>
+          <updateRate>10</updateRate>
+          <imageTopicName>rgb/image_raw</imageTopicName>
+          <depthImageTopicName>depth/image_raw</depthImageTopicName>
+          <pointCloudTopicName>depth/points</pointCloudTopicName>
+          <cameraInfoTopicName>rgb/camera_info</cameraInfoTopicName>
+          <depthImageCameraInfoTopicName>depth/camera_info</depthImageCameraInfoTopicName>
+          <frameName>camera_depth_optical_frame</frameName>
+          <baseline>0.1</baseline>
+          <distortion_k1>0.0</distortion_k1>
+          <distortion_k2>0.0</distortion_k2>
+          <distortion_k3>0.0</distortion_k3>
+          <distortion_t1>0.0</distortion_t1>
+          <distortion_t2>0.0</distortion_t2>
+          <pointCloudCutoff>0.4</pointCloudCutoff>
+        </plugin>
+      </sensor>
+    </gazebo>
+  </xacro:macro>
 </robot>

Commit message: much better Gz behavior through surface tags

File: turtlebot2_description/urdf/kobuki.urdf.xacro (robot description, xacro)
@@ -57,5 +57,4 @@
           <mesh filename="package://kobuki_description/meshes/wheel.dae"/>
         </geometry>
-        <origin xyz="0 0 0" rpy="0 0 0"/>
       </visual>
       <collision>
@@ -63,5 +62,12 @@
           <cylinder length="0.0206" radius="0.035"/>
         </geometry>
-        <origin rpy="0 0 0" xyz="0 0 0"/>
+          <surface>
+            <friction>
+                <ode>
+                    <mu>1</mu>
+                    <mu2>0</mu2>
+                </ode>
+            </friction>
+        </surface>
       </collision>
       <inertial>
@@ -84,5 +90,4 @@
           <mesh filename="package://kobuki_description/meshes/wheel.dae"/>
         </geometry>
-        <origin xyz="0 0 0" rpy="0 0 0"/>
       </visual>
       <collision>
@@ -90,5 +95,12 @@
           <cylinder length="0.0206" radius="0.035"/>
         </geometry>
-        <origin rpy="0 0 0" xyz="0 0 0"/>
+          <surface>
+            <friction>
+                <ode>
+                    <mu>1</mu>
+                    <mu2>0</mu2>
+                </ode>
+            </friction>
+        </surface>
       </collision>
       <inertial>
@@ -108,7 +120,15 @@
       <collision>
         <geometry>
-          <cylinder length="0.0176" radius="0.017"/>
-        </geometry>
-        <origin rpy="0 0 0" xyz="0 0 0"/>
+          <sphere radius="0.017"/>
+<!--           <cylinder length="0.0176" radius="0.017"/> -->
+        </geometry>
+                 <surface>
+            <friction>
+                <ode>
+                    <mu>0</mu>
+                    <mu2>0</mu2>
+                </ode>
+            </friction>
+        </surface>
       </collision>
       <inertial>
@@ -128,7 +148,15 @@
       <collision>
         <geometry>
-          <cylinder length="0.0176" radius="0.017"/>
-        </geometry>
-        <origin rpy="0 0 0" xyz="0 0 0"/>
+          <sphere radius="0.017"/>
+<!--           <cylinder length="0.0176" radius="0.017"/> -->
+        </geometry>
+         <surface>
+            <friction>
+                <ode>
+                    <mu>0</mu>
+                    <mu2>0</mu2>
+                </ode>
+            </friction>
+        </surface>
       </collision>
       <inertial>
@@ -150,5 +178,4 @@
       <inertial>
         <mass value="0.001"/>
-        <origin xyz="0 0 0" rpy="0 0 0"/>
         <inertia ixx="0.0001" ixy="0" ixz="0"
                  iyy="0.000001" iyz="0"
@@ -200,39 +227,13 @@
 <xacro:if value="$(arg gazebo)">
 <gazebo reference="$(arg prefix)wheel_left_link">
-  <mu1>0.1</mu1>
-  <mu2>0.1</mu2>
-  <kp>500000.0</kp>
-  <kd>10.0</kd>
-  <minDepth>0.001</minDepth>
-  <maxVel>0.1</maxVel>
-  <fdir1>1 0 0</fdir1>
   <material>Gazebo/FlatBlack</material>
 </gazebo>
 <gazebo reference="$(arg prefix)wheel_right_link">
-  <mu1>0.1</mu1>
-  <mu2>0.1</mu2>
-  <kp>500000.0</kp>
-  <kd>10.0</kd>
-  <minDepth>0.001</minDepth>
-  <maxVel>0.1</maxVel>
-  <fdir1>1 0 0</fdir1>
   <material>Gazebo/FlatBlack</material>
 </gazebo>
 <gazebo reference="$(arg prefix)caster_back_right_link">
-  <mu1>0.1</mu1>
-  <mu2>0.1</mu2>
-  <kp>1000000.0</kp>
-  <kd>100.0</kd>
-  <minDepth>0.001</minDepth>
-  <maxVel>1.0</maxVel>
   <material>Gazebo/FlatBlack</material>
 </gazebo>
 <gazebo reference="$(arg prefix)caster_back_left_link">
-  <mu1>0.1</mu1>
-  <mu2>0.1</mu2>
-  <kp>1000000.0</kp>
-  <kd>100.0</kd>
-  <minDepth>0.001</minDepth>
-  <maxVel>1.0</maxVel>
   <material>Gazebo/FlatBlack</material>
 </gazebo>
